File: EMUZ80_RP2040.kicad_pcb (KiCad board)
At the start: 2 copper layers, 99.1 x 75.6 mm, 20 parts, among them J1 Conn_01x06_Pin, J2 Conn_01x14_Pin, J3 Conn_01x04_Pin, J4 Conn_01x02_Pin_flat, J6 Conn_02x20_Odd_Even, U1 Z80CPU, U2 AE_RP2040

Commit message: main: AE-RP2040 version Rev001 garber finished
Other:
- board text added: "(C) 2026, N. Kumagai"
- board text added: "[EMUZ80_AE_RP2020] ZILOG Z80 with ROM/RAM/UART Emulator (on AE-RP2040 or compatibles)"
- board text removed: "EMUZ80_AE_RP2020 (C) 2026, N. Kumagai"
